File: electronics/left_main/left_main.kicad_pcb (KiCad board)
At the start: 4 copper layers, 45 x 51 mm, 89 parts, among them IC1 AS3435-EQFM, IC2 AS3435-EQFM, J1 connectors_board, J10 right_side, J11 right_side, J12 right_side, J13 right_side, J14 right_side, J15 right_side, J16 right_side, J17 right_side, J18 right_side, J19 ear_sensor, J20 ear_sensor, J21 ear_sensor, J22 ear_sensor, J23 FB_Filters, J24 FF_Filters, J3 FF_MIC_L_+, J4 FF_MIC_L_-, J5 FB_MIC_L_+, J6 FB_MIC_L_-, J7 HP_L_+, J8 HP_L_-, J9 right_side, SW2 reset_button, U1 BM83, U2 ATSAMD21G18_QFN, U3 MCP73831T-2ACI/OT, U4 SPX3819-3.3, U5 MAX17048G+T10, U6 AP2127K-1.8, U7 AP22814AW5, U8 AP22814AW5, Y1 32.768KHz

Commit message: all pcbs done and ordered
Parts:
- moved J23 2.46 mm to (77.5, 61.0), turned to 0 degrees
Connections:
- net /HP_driver_L/FF_IOP1 renamed /FF_IOP1_L
- net /HP_driver_L/FF_QMIC renamed /FF_QMIC_L
- net /HP_driver_L/FF_QOP1 renamed /FF_QOP1_L
- net /HP_driver_R/FF_IOP1 renamed /FF_IOP1_R
- IC1 pad 16: /HP_driver_R/FB_QMIC -> /FB_QMIC_R
- IC1 pad 17: /HP_driver_R/IOP1R -> /FB_IOP1_R
- IC1 pad 18: /HP_driver_R/QOP1R -> /FB_QOP1_R
- IC1 pad 19: /HP_driver_R/IOP2R -> /FB_IOP2_R
- IC1 pad 20: /HP_driver_R/QOP2R -> /FB_QOP2_R
- IC1 pad 24: /HP_driver_R/FF_QOP1 -> /FF_QOP1_R
- IC1 pad 34: /HP_driver_R/FF_QOP1 -> /FF_QOP1_R
- IC1 pad 36: /HP_driver_R/FF_QMIC -> /FF_QMIC_R
- IC2 pad 16: /HP_driver_L/FB_QMIC -> /FB_QMIC_L
- IC2 pad 17: /HP_driver_L/IOP1R -> /FB_IOP1_L
- IC2 pad 18: /HP_driver_L/QOP1R -> /FB_QOP1_L
- IC2 pad 19: /HP_driver_L/IOP2R -> /FB_IOP2_L
- IC2 pad 20: /HP_driver_L/QOP2R -> /FB_QOP2_L
- J23 pad 10: /HP_driver_L/IOP1R -> /FB_IOP1_R
- J23 pad 11: /HP_driver_L/QOP1R -> /FB_QOP1_R
- J23 pad 12: /HP_driver_L/IOP2R -> /FB_IOP2_R
- J23 pad 13: /HP_driver_L/QOP2R -> /FB_QOP2_R
- J23 pad 2: /HP_driver_R/FB_QMIC -> /FB_QMIC_L
- J23 pad 3: /HP_driver_R/IOP1R -> /FB_IOP1_L
- J23 pad 4: /HP_driver_R/QOP1R -> /FB_QOP1_L
- J23 pad 5: /HP_driver_R/IOP2R -> /FB_IOP2_L
- J23 pad 6: /HP_driver_R/QOP2R -> /FB_QOP2_L
- J23 pad 9: /HP_driver_L/FB_QMIC -> /FB_QMIC_R
- J24 pad 10: /HP_driver_R/FF_QOP1 -> /FF_QMIC_R
- J24 pad 12: /HP_driver_R/FF_QMIC -> /FF_QOP1_R
Routing:
- net /HP_driver_L/QOP2R: track 40.0 -> 0.00 mm, vias 1 -> 0
- net /HP_driver_L/IOP2R: track 39.0 -> 0.00 mm, vias 1 -> 0
- net /HP_driver_L/FB_QMIC: track 39.0 -> 0.00 mm, vias 1 -> 0
- net /HP_driver_L/IOP1R: track 39.0 -> 0.00 mm, vias 1 -> 0
- net /HP_driver_L/QOP1R: track 38.7 -> 0.00 mm, vias 1 -> 0
- net /FB_QOP2_L: track 0.00 -> 36.3 mm, vias 0 -> 1
- net /FB_IOP2_L: track 0.00 -> 34.4 mm, vias 0 -> 1
- net /FB_QOP1_L: track 0.00 -> 33.2 mm, vias 0 -> 1
- net /FB_IOP1_L: track 0.00 -> 32.7 mm, vias 0 -> 1
- net /FB_QMIC_L: track 0.00 -> 31.8 mm, vias 0 -> 1
- net /HP_driver_R/FF_QOP1: track 30.5 -> 0.00 mm, vias 3 -> 0
- net /FF_QOP1_R: track 0.00 -> 28.9 mm, vias 0 -> 3
- net /HP_driver_R/FF_QMIC: track 18.4 -> 0.00 mm, vias 1 -> 0
- net /FF_QMIC_R: track 0.00 -> 17.4 mm, vias 0 -> 1
- net /FB_IOP2_R: track 0.00 -> 10.7 mm, vias 0 -> 1
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Other:
- board text added: "FB filter pcb"
- board text added: "FF filter pcb"
