File: electronics/left_main/left_main.kicad_sch (KiCad schematic)
At the start: 23 parts, among them J1 Conn_01x18_Pin, SW1 SPST_TACT-KMR2, U1 BM83, U2 ATSAMD21G18_QFN, U3 MCP73831T-2ACI/OT, U4 SPX3819-3.3, X1 32.768

Commit message: schematic done, blocks located, uC1 + PWR routed
Parts:
- removed C1, C6, C7, C8: 10uF, Capacitor_SMD:C_0402_1005Metric, symbol Adafruit Feather M0 Basic rev C-eagle-import:CAP_CERAMIC0805-NOOUTLINE
- removed C2, C3: 1uF, Capacitor_SMD:C_0402_1005Metric, symbol Adafruit Feather M0 Basic rev C-eagle-import:CAP_CERAMIC0603_NO
- removed C4, C5: 22pF, Capacitor_SMD:C_0402_1005Metric, symbol Adafruit Feather M0 Basic rev C-eagle-import:CAP_CERAMIC0603_NO
- removed CHG1: ORANGE, LED_SMD:LED_0603_1608Metric, symbol Adafruit Feather M0 Basic rev C-eagle-import:LED0805_NOOUTLINE
- removed J1: Conn_01x18_Pin, symbol Connector:Conn_01x18_Pin
- removed R1: 2.2K, Resistor_SMD:R_0402_1005Metric, symbol Adafruit Feather M0 Basic rev C-eagle-import:RESISTOR_0603_NOOUT
- removed R2: 100k, Resistor_SMD:R_0402_1005Metric, symbol Adafruit Feather M0 Basic rev C-eagle-import:RESISTOR_0603_NOOUT
- removed R3: 100K, Resistor_SMD:R_0402_1005Metric, symbol Adafruit Feather M0 Basic rev C-eagle-import:RESISTOR_0603_NOOUT
- removed R4: 1K, Resistor_SMD:R_0402_1005Metric, symbol Adafruit Feather M0 Basic rev C-eagle-import:RESISTOR_0603_NOOUT
- removed R5: 10K, Resistor_SMD:R_0402_1005Metric, symbol Adafruit Feather M0 Basic rev C-eagle-import:RESISTOR_0603_NOOUT
- removed SW1: SPST_TACT-KMR2, Button_Switch_SMD:SW_Push_1P1T_NO_CK_KMR2, symbol Adafruit Feather M0 Basic rev C-eagle-import:SPST_TACT-KMR2
- removed X1: 32.768, other footprints:XTAL3215, symbol Adafruit Feather M0 Basic rev C-eagle-import:XTAL-3.2X1.5
- added C1, C4, C6, C7, C8: 10uF, Capacitor_SMD:C_0402_1005Metric_Pad0.74x0.62mm_HandSolder, symbol Device:C_Small
- added C2, C3, C75, C76, C77: 1uF, Capacitor_SMD:C_0402_1005Metric_Pad0.74x0.62mm_HandSolder, symbol Device:C_Small
- added C4, C5: 22pF, Capacitor_SMD:C_0402_1005Metric_Pad0.74x0.62mm_HandSolder, symbol Device:C_Small
- added C5: 0.1uF, Capacitor_SMD:C_0402_1005Metric_Pad0.74x0.62mm_HandSolder, symbol Device:C_Small
- added J10, J11, J12, J13, J14, J15, J16, J17, J18, J9: right_side, TestPoint:TestPoint_Pad_D1.0mm, symbol Connector:TestPoint
- added J19, J20, J21: ear_sensor, TestPoint:TestPoint_Pad_D1.0mm, symbol Connector:TestPoint
- added J3: FF_MIC_L_+, TestPoint:TestPoint_Pad_D1.0mm, symbol Connector:TestPoint
- added J3: connectors_board, SFV18R-1STE1LF:CON18_1X18_DR_SFV_GLE, symbol Connector:Conn_01x18_Pin
- added J4: FF_MIC_L_-, TestPoint:TestPoint_Pad_D1.0mm, symbol Connector:TestPoint
- added J5: FB_MIC_L_+, TestPoint:TestPoint_Pad_D1.0mm, symbol Connector:TestPoint
- added J6: FB_MIC_L_-, TestPoint:TestPoint_Pad_D1.0mm, symbol Connector:TestPoint
- added J7: HP_L_+, TestPoint:TestPoint_Pad_D1.0mm, symbol Connector:TestPoint
- added J8: HP_L_-, TestPoint:TestPoint_Pad_D1.0mm, symbol Connector:TestPoint
- added OC1: Optocoupler_Generic, x, symbol PCM_Optocoupler_AKL:Optocoupler_Generic
- added R1: 2.2k, Resistor_SMD:R_0402_1005Metric_Pad0.72x0.64mm_HandSolder, symbol Device:R
- added R2, R3, R5: 100k, Resistor_SMD:R_0402_1005Metric_Pad0.72x0.64mm_HandSolder, symbol Device:R
- added R2: 68k, Resistor_SMD:R_0402_1005Metric_Pad0.72x0.64mm_HandSolder, symbol Device:R
- added R3: 200, Resistor_SMD:R_0402_1005Metric_Pad0.72x0.64mm_HandSolder, symbol Device:R
- added R4: 6.8K, Resistor_SMD:R_0402_1005Metric_Pad0.72x0.64mm_HandSolder, symbol Device:R
- added SW2: reset_button, Button_Switch_SMD:SW_Push_1P1T_NO_CK_KMR2, symbol Switch:SW_SPST
- added U2 (x2): AP22814AW5, Package_TO_SOT_SMD:SOT-23-5, symbol Power_Management:AP22814AW5
- added U5: MAX17048G+T10, MAX17048G+T10:21-0168E_T822-3_MXM, symbol MAX17048:MAX17048G+T10
- added U6: AP2127K-1.8, Package_TO_SOT_SMD:SOT-23-5, symbol Regulator_Linear:AP2127K-1.8
- added Y1: 32.768KHz, Crystal:Crystal_SMD_3215-2Pin_3.2x1.5mm, symbol Device:Crystal_Small
Connections:
- net BAT_IN is gone; now on net +3V3: U1.23 (BAT_IN)
- net P3_4 is gone; now on net BM83_PROG_EN: U1.31 (P3_4/UART_RTS)
- net PWR(MFB) is gone; now on net D4: U1.26 (PWR(MFB))
- net +3V3: now also C1.1, C4.1, C75.1, J17.1, J3.17 (Pin_17), U2.1 (OUT), U2.5 (IN), U6.1 (VIN), U6.3 (EN); no longer U2.17 (VDDIO), U2.36 (VDDIO), U2.44 (VDDIN), U2.6 (VDDA)
- net +BATT: now also C6.1, J16.1, R2.1, U5.2 (CELL), U5.3 (VDD)
- net A3: now also U2.4 (EN)
- net A4: now also J21.1, OC1.3, R2.1
- net AREF: now also C77.1
- net D10: now also J3.13 (Pin_13)
- net D11: now also J3.4 (Pin_4)
- net D13: now also R1.1
- net D2: now also J3.9 (Pin_9)
- net D3: now also J15.1
- net GND: now also C1.2, C2.2, C3.2, C4.1, C4.2, C5.1, C5.2, C6.2, C7.2, C75.2, C76.2, C77.2, C8.2, J18.1, J3.1 (Pin_1), J3.16 (Pin_16), R2.2, R3.2, R3.2, R4.2, SW2.2 (B), U2.2 (GND), U2.2 (GND), U5.1 (CTG), U5.4 (GND), U5.6 (QSTRT), U5.9 (EPAD), U6.2 (GND)
- net VBUS: now also C7.1, J3.18 (Pin_18); no longer U1.22 (ADAP_IN)
- net ~{RESET}: now also R5.2, SW2.1 (A)
- net at U2.43 (VDDCORE): now also C3.1
- net VDD: now reaches U4.5 (OUT)
- net VDD: now also U2.17 (VDDIO), U2.36 (VDDIO), U2.44 (VDDIN), U2.6 (VDDA), C2.1, C8.1, R5.1, U2.5 (IN)
- net at U2.2 (PA01/EINT1/SERCOM1.1): now also C5.2, Y1.2
- net at D1.2 (A): now also R1.2
- net at U2.1 (PA00/EINT0/SERCOM1.0): now also C4.2, Y1.1
- net at U3.5 (PROG): now also R4.1
- net CHRG_STAT renamed BM83_PROG_EN
- net D+ renamed USB_D+
- net USB_D+: now also J3.14 (Pin_14)
- net D- renamed USB_D-
- net USB_D-: now also J3.15 (Pin_15)
- net D12 renamed ANC_ON
- net ANC_ON: now also J3.12 (Pin_12)
- net D5 renamed 3V3_EN
- net 3V3_EN: now also U2.4 (EN)
- net D6 renamed ANC_OFF
- net ANC_OFF: now also J3.11 (Pin_11)
- net D7 renamed ANC_PBO
- net ANC_PBO: now also J3.10 (Pin_10)
- net D9 renamed BAT_V_SENSE
- net BAT_V_SENSE: now also R2.2, R3.1
- net SCL renamed I2C_SCL
- net I2C_SCL: now also U5.7 (SCL)
- net SDA renamed I2C_SDA
- net I2C_SDA: now also U5.8 (SDA)
- new net: J20.1, OC1.2, R3.1
- new net: C5.1, J19.1, OC1.1, OC1.4, U2.1 (OUT)
- new net +1V8: C76.1, U6.5 (VOUT)
- new net ADAP_IN: U1.22 (ADAP_IN)
- new net FB_mic_L_+: J5.1
- new net FB_mic_L_-: J6.1
- new net FB_mic_R_+: J11.1
- new net FB_mic_R_-: J12.1
- new net FF_mic_L_+: J3.1
- new net FF_mic_L_-: J4.1
- new net FF_mic_R_+: J9.1
- new net FF_mic_R_-: J10.1
- new net HP_L_+: J7.1
- new net HP_L_-: J8.1
- new net HP_R_+: J13.1
- new net HP_R_-: J14.1
- new net audio_in_L: J3.2 (Pin_2)
- new net audio_in_R: J3.3 (Pin_3)
- no-connect marks 0 -> 55
Other:
- added sheet HP_driver_L (ANC_HP_Driver.kicad_sch)
- sheet HP_driver_R ports: added FB_mic_+, FB_mic_-, FF_mic_+, FF_mic_-, HP_+, HP_-, bypass_in, i2c_clk, i2c_sda, line_in, vneg; removed none
- note added: "6.8K = 150mA 6 hr charge time with 935mAh battery"
- note added: "ANC Headphone Drivers (4)"
- note added: "BM83 BTM (7)"
- note added: "Battery Charging and Monitoring (1)"
- note added: "Connectors"
- note added: "Ear sensor L (3)"
- note added: "I(mA) = 1000V/R_Prog(kOhm)"
- note added: "Power Supplies (2)"
- note added: "SAMD21 MCU (6)"
- note added: "close to battery -ve terminal"
- note added: "sensor connected on the other end of wires on tp19-21"
- note added: "swapping clk and data for two i2c addresses"
- note added: "taken from a feather m0, so it's best to try to only use pins exposed by the board"
- note added: "~{Buttons}"
- note added: "~{sensing}"
- note added: "~{serials}"
- note removed: "1.0K = 1000mA"
- note removed: "10K = 100mA"
- note removed: "2.0K = 500mA"
- note removed: "3.3v supply"
- note removed: "5.0K = 200mA"
- note removed: "BM83 BTM (3)"
- note removed: "SAMD21 MCU (1)"
- note removed: "USB AND BATTERY CHARGING"
- moved on the sheet: D1, D2, U1, U2, U3, U4

Commit message: oops forgot to save and close
Connections:
- no-connect marks 55 -> 54
Other:
- note added: "No separate ground planes are used, instead, analogue and digital areas of one plane are used"
Changed lines of the file:
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@@
   (no_connect (at 318.77 160.02))
   (no_connect (at 34.29 68.58))
-  (no_connect (at 384.81 154.94))
   (no_connect (at 318.77 203.2))
   (no_connect (at 384.81 182.88))
@@
   (no_connect (at 318.77 177.8))
   (no_connect (at 384.81 208.28))
-  (wire (pts (xy 49.53 185.42) (xy 49.53 187.96))
+  (wire (pts (xy 48.26 185.42) (xy 48.26 187.96))
     (stroke (width 0) (type default))
   )
@@
   )
   (wire (pts (xy 163.83 251.46) (xy 181.61 251.46))
+    (stroke (width 0) (type default))
+  )
+  (wire (pts (xy 48.26 185.42) (xy 49.53 185.42))
     (stroke (width 0) (type default))
   )
@@
   (text "ANC Headphone Drivers (4)" (at 302.26 20.32 0)
     (effects (font (size 3 3)) (justify left bottom))
+  )
+  (text "No separate ground planes are used, instead, \nanalogue and digital areas of one plane are used"
+    (at 147.32 140.97 0)
+    (effects (font (size 1.27 1.27)) (justify left bottom))
   )
   (text "~{sensing}" (at 203.2 200.66 90)
@@
     )
   )
-  (symbol (lib_id "power:GND") (at 49.53 187.96 0) (mirror y) (unit 1)
-    (in_bom yes) (on_board yes) (dnp no) (fields_autoplaced)
-    (property "Reference" "#PWR06" (at 49.53 194.31 0)
-      (effects (font (size 1.27 1.27)) hide)
-    )
-    (property "Value" "GND" (at 49.53 192.405 0)
-      (effects (font (size 1.27 1.27)))
-    )
-    (property "Footprint" "" (at 49.53 187.96 0)
-      (effects (font (size 1.27 1.27)) hide)
-    )
-    (property "Datasheet" "" (at 49.53 187.96 0)
-      (effects (font (size 1.27 1.27)) hide)
-    )
+  (symbol (lib_id "power:GND") (at 48.26 187.96 0) (mirror y) (unit 1)
+    (in_bom yes) (on_board yes) (dnp no) (fields_autoplaced)
+    (property "Reference" "#PWR06" (at 48.26 194.31 0)
+      (effects (font (size 1.27 1.27)) hide)
+    )
+    (property "Value" "GND" (at 48.26 192.405 0)
+      (effects (font (size 1.27 1.27)))
+    )
+    (property "Footprint" "" (at 48.26 187.96 0)
+      (effects (font (size 1.27 1.27)) hide)
+    )
+    (property "Datasheet" "" (at 48.26 187.96 0)
+      (effects (font (size 1.27 1.27)) hide)
+    )

Commit message: L filterers + drivers layout
Parts:
- added R74, R75: 10k, Resistor_SMD:R_0402_1005Metric_Pad0.72x0.64mm_HandSolder, symbol Device:R
- J3: symbol Connector:Conn_01x18_Pin -> Connector:Conn_01x20_Pin
Connections:
- net ANC_OFF: now also J3.13 (Pin_13); no longer J3.11 (Pin_11)
- net ANC_ON: now also J3.14 (Pin_14); no longer J3.12 (Pin_12)
- net ANC_PBO: now also J3.12 (Pin_12); no longer J3.10 (Pin_10)
- net D10: now also J3.15 (Pin_15); no longer J3.13 (Pin_13)
- net D2: now also J3.11 (Pin_11); no longer J3.9 (Pin_9)
- net GND: now also J3.19 (Pin_19), J3.20 (Pin_20)
- net I2C_SCL: now also R74.2
- net I2C_SDA: now also R75.2
- net USB_D+: now also J3.9 (Pin_9); no longer J3.14 (Pin_14)
- net USB_D-: now also J3.10 (Pin_10); no longer J3.15 (Pin_15)
- net VDD: now also R74.1, R75.1
Other:
- note added: "EP"

Commit message: drc happy, silkscreens everywhere
Parts:
- added J22: ear_sensor, TestPoint:TestPoint_Pad_D1.0mm, symbol Connector:TestPoint
Connections:
- net A2: now also OC1.4, J22.1
- net at C5.1, J19.1, OC1.1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: no longer OC1.4
Other:
- note removed: "sensor connected on the other end of wires on tp19-21"
Changed lines of the file:
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@@
   (junction (at 62.23 35.56) (diameter 0) (color 0 0 0 0)
   )
+  (junction (at 266.7 82.55) (diameter 0) (color 0 0 0 0)
+  )
   (junction (at 82.55 190.5) (diameter 0) (color 0 0 0 0)
   )
@@
     (stroke (width 0) (type default))
   )
+  (wire (pts (xy 266.7 78.74) (xy 275.59 78.74))
+    (stroke (width 0) (type default))
+  )
   (wire (pts (xy 208.28 60.96) (xy 208.28 50.8))
     (stroke (width 0) (type default))
@@
     (stroke (width 0) (type default))
   )
-  (wire (pts (xy 266.7 82.55) (xy 266.7 78.74))
-    (stroke (width 0) (type default))
-  )
   (wire (pts (xy 138.43 119.38) (xy 138.43 123.19))
     (stroke (width 0) (type default))
@@
     (stroke (width 0) (type default))
   )
-  (wire (pts (xy 266.7 78.74) (xy 259.08 78.74))
-    (stroke (width 0) (type default))
-  )
   (wire (pts (xy 163.83 236.22) (xy 181.61 236.22))
     (stroke (width 0) (type default))
@@
     (stroke (width 0) (type default))
   )
+  (wire (pts (xy 266.7 82.55) (xy 266.7 78.74))
+    (stroke (width 0) (type default))
+  )
   (wire (pts (xy 266.7 57.15) (xy 266.7 58.42))
     (stroke (width 0) (type default))
@@
     (effects (font (size 3 3)) (justify left bottom))
   )
-  (text "sensor connected on the other \nend of wires on tp19-21"
-    (at 267.97 80.01 0)
-    (effects (font (size 1.27 1.27)) (justify left bottom))
-  )
   (text "EP" (at 35.56 33.02 0)
     (effects (font (size 1.27 1.27)) (justify left bottom))
@@
     (effects (font (size 1.2446 1.2446)) (justify left bottom))
   )
+  (label "A2" (at 269.24 78.74 0) (fields_autoplaced)
+    (effects (font (size 1.2446 1.2446)) (justify left bottom))
+  )
   (label "ANC_OFF" (at 181.61 238.76 0) (fields_autoplaced)
     (effects (font (size 1.27 1.27)) (justify left bottom))
@@
         )
       )
+    )
+  )
+  (symbol (lib_id "Connector:TestPoint") (at 266.7 82.55 270) (unit 1)
+    (in_bom yes) (on_board yes) (dnp no)
+    (property "Reference" "J22" (at 273.05 81.28 90)
+      (effects (font (size 1.27 1.27)))
+    )
+    (property "Value" "ear_sensor" (at 270.002 84.2739 90)
+      (effects (font (size 1.27 1.27)) hide)
+    )
+    (property "Footprint" "TestPoint:TestPoint_Pad_D1.0mm" (at 266.7 87.63 0)
+      (effects (font (size 1.27 1.27)) hide)
+    )
+    (property "Datasheet" "~" (at 266.7 87.63 0)
+      (effects (font (size 1.27 1.27)) hide)
+    )
+    (pin "1")
+    (instances
+      (project "left_main"
+        (path "/7f46bcb9-0051-4f2d-b9e2-7f7ba1d1d684"
+          (reference "J22") (unit 1)
+        )
+      )

Commit message: FB,FF filter separated from main schematic
Parts:
- added J23: FB_Filters, Connector_Hirose:Hirose_DF12_DF12E3.0-14DP-0.5V_2x07_P0.50mm_Vertical, symbol Connector:Conn_01x14_Pin
- added J24: FF_Filters, Connector_Hirose:Hirose_DF12_DF12E3.0-14DP-0.5V_2x07_P0.50mm_Vertical, symbol Connector:Conn_01x14_Pin
Connections:
- net GND: now also J23.1 (Pin_1), J23.14 (Pin_14), J23.7 (Pin_7), J23.8 (Pin_8), J24.1 (Pin_1), J24.13 (Pin_13), J24.14 (Pin_14), J24.2 (Pin_2), J24.6 (Pin_6), J24.7 (Pin_7), J24.8 (Pin_8), J24.9 (Pin_9)
- new net HP_driver_L/FB_IOP1: J23.10 (Pin_10)
- new net HP_driver_L/FB_IOP2: J23.12 (Pin_12)
- new net HP_driver_L/FB_QMIC: J23.9 (Pin_9)
- new net HP_driver_L/FB_QOP1: J23.11 (Pin_11)
- new net HP_driver_L/FB_QOP2: J23.13 (Pin_13)
- new net HP_driver_L/FF_IOP1: J24.4 (Pin_4)
- new net HP_driver_L/FF_QMIC: J24.5 (Pin_5)
- new net HP_driver_L/FF_QOP1: J24.3 (Pin_3)
- new net HP_driver_R/FB_IOP1: J23.3 (Pin_3)
- new net HP_driver_R/FB_IOP2: J23.5 (Pin_5)
- new net HP_driver_R/FB_QMIC: J23.2 (Pin_2)
- new net HP_driver_R/FB_QOP1: J23.4 (Pin_4)
- new net HP_driver_R/FB_QOP2: J23.6 (Pin_6)
- new net HP_driver_R/FF_IOP1: J24.11 (Pin_11)
- new net HP_driver_R/FF_QMIC: J24.12 (Pin_12)
- new net HP_driver_R/FF_QOP1: J24.10 (Pin_10)
Other:
- sheet HP_driver_L ports: added FB_IOP1, FB_IOP2, FB_QMIC, FB_QOP1, FB_QOP2, FF_IOP1, FF_QMIC, FF_QOP1; removed none
- sheet HP_driver_R ports: added FB_IOP1, FB_IOP2, FB_QMIC, FB_QOP1, FB_QOP2, FF_IOP1, FF_QMIC, FF_QOP1; removed none
- moved on the sheet: C1, C2, C3, C4, C5, C77, D1, J19, J20, J21, J22, OC1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

Commit message: all pcbs done and ordered
Connections:
- net HP_driver_L/FB_IOP1 renamed FB_IOP1_R
- net HP_driver_L/FB_IOP2 renamed FB_IOP2_R
- net HP_driver_L/FB_QMIC renamed FB_QMIC_R
- net HP_driver_L/FB_QOP1 renamed FB_QOP1_R
- net HP_driver_L/FB_QOP2 renamed FB_QOP2_R
- net HP_driver_L/FF_IOP1 renamed FF_IOP1_L
- net HP_driver_L/FF_QMIC renamed FF_QMIC_L
- net HP_driver_L/FF_QOP1 renamed FF_QOP1_L
- net HP_driver_R/FB_IOP1 renamed FB_IOP1_L
- net HP_driver_R/FB_IOP2 renamed FB_IOP2_L
- net HP_driver_R/FB_QMIC renamed FB_QMIC_L
- net HP_driver_R/FB_QOP1 renamed FB_QOP1_L
- net HP_driver_R/FB_QOP2 renamed FB_QOP2_L
- net HP_driver_R/FF_IOP1 renamed FF_IOP1_R
- net HP_driver_R/FF_QMIC renamed FF_QOP1_R
- net HP_driver_R/FF_QOP1 renamed FF_QMIC_R
Other:
- moved on the sheet: J23, J24
