File: electronics/left_main/FF_Filter_PCB/FF_Filter_PCB.kicad_pcb (KiCad board)
At the start: 4 copper layers, 35 parts, among them J1 FF_Filters

Commit message: FF filter PCB done
Parts:
- C1, C10, C11, C12, C13, C14, C15, C16, C2, C3, C4, C5, C6, C7, C8, C9, J1, R1, R10, R11, R12, R13, R14, R15, R16, R17, R18, R2, R3, R4, R5, R6, R7, R8, R9: moved to B.Cu
- moved C16 33.2 mm to (79.4, 50.6), turned to 90 degrees
- moved R18 29.5 mm to (80.3, 54.2)
- moved C14 29.4 mm to (78.3, 53.5), turned to -90 degrees
- moved R16 28.8 mm to (80.9, 50.6), turned to -90 degrees
- moved C10 28.2 mm to (78.3, 47.7), turned to 90 degrees
- moved C15 26.7 mm to (83.0, 54.2), turned to 180 degrees
- moved R15 26.1 mm to (80.3, 52.7), turned to 180 degrees
- moved R17 25.7 mm to (85.0, 53.5), turned to 90 degrees
- moved C11 25.2 mm to (83.0, 48.4), turned to 180 degrees
- moved C13 25.0 mm to (83.0, 52.7)
- moved R12 24.9 mm to (80.3, 48.4)
- moved C12 24.5 mm to (84.5, 49.9)
- moved C9 23.6 mm to (83.0, 46.9)
- moved R13 23.3 mm to (82.4, 50.6), turned to 90 degrees
- moved R10 23.3 mm to (80.3, 46.9), turned to 180 degrees
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Routing:
- net /filter_L/IOP1: track 0.00 -> 20.5 mm
- net /filter_R/IOP1: track 0.00 -> 17.5 mm
- net /filter_L/QMIC: track 0.00 -> 14.4 mm
- net /filter_L/QOP1: track 0.00 -> 12.5 mm
- net /filter_R/QMIC: track 0.00 -> 11.5 mm
- net /filter_R/QOP1: track 0.00 -> 9.70 mm
- net Net-(C7-Pad2): track 0.00 -> 5.16 mm
- net Net-(C15-Pad2): track 0.00 -> 5.16 mm
- net Net-(C3-Pad2): track 0.00 -> 4.61 mm
- net Net-(C11-Pad2): track 0.00 -> 4.61 mm
- net Net-(C5-Pad2): track 0.00 -> 3.00 mm
- net Net-(C13-Pad2): track 0.00 -> 3.00 mm
- net Net-(C11-Pad1): track 0.00 -> 3.00 mm
- net Net-(C1-Pad2): track 0.00 -> 3.00 mm
- net Net-(C6-Pad1): track 0.00 -> 2.98 mm
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- added copper zone on B.Cu, net GNDA
Other:
- board outline added: 18 x 20.1 mm

Commit message: all pcbs done and ordered
Parts:
- J1: footprint Connector_Hirose:Hirose_DF12_DF12E3.0-14DP-0.5V_2x07_P0.50mm_Vertical -> Connector_Hirose:Hirose_DF12_DF12C3.0-14DS-0.5V_2x07_P0.50mm_Vertical
- moved C1 1.14 mm to (81.9, 55.9)
- moved C10 1.14 mm to (77.2, 47.7)
- moved C11 1.14 mm to (81.9, 48.4)
- moved C12 1.14 mm to (83.3, 49.9)
- moved C13 1.14 mm to (81.9, 52.7)
- moved C14 1.14 mm to (77.2, 53.5)
- moved C15 1.14 mm to (81.9, 54.2)
- moved C16 1.14 mm to (78.3, 50.6)
- moved C2 1.14 mm to (77.1, 56.6)
- moved C3 1.14 mm to (81.9, 57.4)
- moved C4 1.14 mm to (83.3, 58.9)
- moved C5 1.14 mm to (81.9, 61.7)
- moved C6 1.14 mm to (77.1, 62.4)
- moved C7 1.14 mm to (81.9, 63.2)
- moved C8 1.14 mm to (78.2, 59.5)
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Connections:
- J1 pad 10: /filter_R/QOP1 -> /filter_R/QMIC
- J1 pad 12: /filter_R/QMIC -> /filter_R/QOP1
Routing:
- net /filter_L/QOP1: track 12.5 -> 7.93 mm
- net /filter_L/IOP1: track 20.5 -> 17.2 mm
- net /filter_L/QMIC: track 14.4 -> 12.5 mm
- net /filter_R/QMIC: track 11.5 -> 10.3 mm
- net /filter_R/IOP1: track 17.5 -> 16.3 mm
- net /filter_R/QOP1: track 9.70 -> 8.63 mm
Other:
- board size 18 x 20.1 mm -> 16.5 x 19.2 mm
- board text added: "FF Filter PCB V0.0"
- board text added: "L"
- board text added: "R"
