File: electronics/left_main/FF_Filter_PCB/FF_Filter_PCB.kicad_sch (KiCad schematic)
At the start: 1 part, among them J1 FF_Filters

Commit message: all pcbs done and ordered
Parts:
- J1: footprint Connector_Hirose:Hirose_DF12_DF12E3.0-14DP-0.5V_2x07_P0.50mm_Vertical -> Connector_Hirose:Hirose_DF12_DF12C3.0-14DS-0.5V_2x07_P0.50mm_Vertical
Connections:
- net filter_R/QMIC: now also J1.10 (Pin_10); no longer J1.12 (Pin_12)
- net filter_R/QOP1: now also J1.12 (Pin_12); no longer J1.10 (Pin_10)
Changed lines of the file:
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@@
   (junction (at 77.47 60.96) (diameter 0) (color 0 0 0 0)
   )
-  (junction (at 104.14 73.66) (diameter 0) (color 0 0 0 0)
+  (junction (at 104.14 82.55) (diameter 0) (color 0 0 0 0)
   )
   (junction (at 77.47 63.5) (diameter 0) (color 0 0 0 0)
@@
   (junction (at 77.47 55.88) (diameter 0) (color 0 0 0 0)
   )
-  (wire (pts (xy 74.93 50.8) (xy 105.41 50.8))
+  (wire (pts (xy 100.33 59.69) (xy 105.41 59.69))
+    (stroke (width 0) (type default))
+  )
+  (wire (pts (xy 97.79 53.34) (xy 97.79 57.15))
+    (stroke (width 0) (type default))
+  )
+  (wire (pts (xy 105.41 62.23) (xy 102.87 62.23))
     (stroke (width 0) (type default))
   )
@@
     (stroke (width 0) (type default))
   )
+  (wire (pts (xy 85.09 71.12) (xy 74.93 71.12))
+    (stroke (width 0) (type default))
+  )
   (wire (pts (xy 77.47 63.5) (xy 77.47 73.66))
     (stroke (width 0) (type default))
@@
     (stroke (width 0) (type default))
   )
-  (wire (pts (xy 74.93 66.04) (xy 105.41 66.04))
+  (wire (pts (xy 102.87 48.26) (xy 74.93 48.26))
+    (stroke (width 0) (type default))
+  )
+  (wire (pts (xy 90.17 74.93) (xy 105.41 74.93))
     (stroke (width 0) (type default))
   )
@@
     (stroke (width 0) (type default))
   )
-  (wire (pts (xy 104.14 55.88) (xy 104.14 73.66))
+  (wire (pts (xy 104.14 64.77) (xy 104.14 82.55))
     (stroke (width 0) (type default))
   )
@@
     (stroke (width 0) (type default))
   )
+  (wire (pts (xy 87.63 68.58) (xy 74.93 68.58))
+    (stroke (width 0) (type default))
+  )
   (wire (pts (xy 74.93 58.42) (xy 77.47 58.42))
     (stroke (width 0) (type default))
@@
     (stroke (width 0) (type default))
   )
-  (wire (pts (xy 74.93 48.26) (xy 105.41 48.26))
-    (stroke (width 0) (type default))
-  )
   (wire (pts (xy 77.47 80.01) (xy 77.47 76.2))
     (stroke (width 0) (type default))
   )
-  (wire (pts (xy 74.93 71.12) (xy 105.41 71.12))
-    (stroke (width 0) (type default))
-  )
-  (wire (pts (xy 74.93 53.34) (xy 105.41 53.34))
+  (wire (pts (xy 85.09 80.01) (xy 105.41 80.01))
+    (stroke (width 0) (type default))
+  )
+  (wire (pts (xy 85.09 80.01) (xy 85.09 71.12))
     (stroke (width 0) (type default))
   )
@@
     (stroke (width 0) (type default))
   )
-  (wire (pts (xy 74.93 68.58) (xy 105.41 68.58))
-    (stroke (width 0) (type default))
-  )
-  (wire (pts (xy 104.14 73.66) (xy 105.41 73.66))
-    (stroke (width 0) (type default))
-  )
-  (wire (pts (xy 105.41 55.88) (xy 104.14 55.88))
-    (stroke (width 0) (type default))
-  )
-  (wire (pts (xy 104.14 80.01) (xy 104.14 73.66))
+  (wire (pts (xy 87.63 77.47) (xy 105.41 77.47))
+    (stroke (width 0) (type default))
+  )
+  (wire (pts (xy 87.63 77.47) (xy 87.63 68.58))
+    (stroke (width 0) (type default))
+  )
+  (wire (pts (xy 104.14 82.55) (xy 105.41 82.55))
+    (stroke (width 0) (type default))
+  )
+  (wire (pts (xy 90.17 66.04) (xy 74.93 66.04))
+    (stroke (width 0) (type default))
+  )
+  (wire (pts (xy 100.33 50.8) (xy 74.93 50.8))
+    (stroke (width 0) (type default))
+  )
+  (wire (pts (xy 105.41 64.77) (xy 104.14 64.77))
+    (stroke (width 0) (type default))
+  )
+  (wire (pts (xy 104.14 88.9) (xy 104.14 82.55))
+    (stroke (width 0) (type default))
+  )
+  (wire (pts (xy 102.87 62.23) (xy 102.87 48.26))
+    (stroke (width 0) (type default))
+  )
+  (wire (pts (xy 90.17 74.93) (xy 90.17 66.04))
+    (stroke (width 0) (type default))
+  )
+  (wire (pts (xy 97.79 57.15) (xy 105.41 57.15))
+    (stroke (width 0) (type default))
+  )
+  (wire (pts (xy 74.93 53.34) (xy 97.79 53.34))
     (stroke (width 0) (type default))
   )
@@
   )
   (wire (pts (xy 77.47 58.42) (xy 77.47 60.96))
+    (stroke (width 0) (type default))
+  )
+  (wire (pts (xy 100.33 59.69) (xy 100.33 50.8))
     (stroke (width 0) (type default))
   )
@@
       (effects (font (size 1.27 1.27)) (justify right))
     )
-    (property "Footprint" "Connector_Hirose:Hirose_DF12_DF12E3.0-14DP-0.5V_2x07_P0.50mm_Vertical" (at 69.85 60.96 0)
+    (property "Footprint" "Connector_Hirose:Hirose_DF12_DF12C3.0-14DS-0.5V_2x07_P0.50mm_Vertical" (at 69.85 60.96 0)
       (effects (font (size 1.27 1.27)) hide)
     )
@@
     )
   )
-  (symbol (lib_id "power:GNDA") (at 104.14 80.01 0) (unit 1)
+  (symbol (lib_id "power:GNDA") (at 104.14 88.9 0) (unit 1)
     (in_bom yes) (on_board yes) (dnp no) (fields_autoplaced)
-    (property "Reference" "#PWR08" (at 104.14 86.36 0)
-      (effects (font (size 1.27 1.27)) hide)
-    )
-    (property "Value" "GNDA" (at 104.14 85.09 0)
+    (property "Reference" "#PWR08" (at 104.14 95.25 0)
+      (effects (font (size 1.27 1.27)) hide)
+    )
+    (property "Value" "GNDA" (at 104.14 93.98 0)
       (effects (font (size 1.27 1.27)))
     )
-    (property "Footprint" "" (at 104.14 80.01 0)
-      (effects (font (size 1.27 1.27)) hide)
-    )
-    (property "Datasheet" "" (at 104.14 80.01 0)
+    (property "Footprint" "" (at 104.14 88.9 0)
+      (effects (font (size 1.27 1.27)) hide)
+    )
+    (property "Datasheet" "" (at 104.14 88.9 0)
       (effects (font (size 1.27 1.27)) hide)
     )
@@
     )
   )
-  (sheet (at 105.41 45.72) (size 29.21 12.7) (fields_autoplaced)
+  (sheet (at 105.41 54.61) (size 29.21 12.7) (fields_autoplaced)
     (stroke (width 0.1524) (type solid))
     (fill (color 0 0 0 0.0000))
-    (property "Sheetname" "filter_R" (at 105.41 45.0084 0)
+    (property "Sheetname" "filter_R" (at 105.41 53.8984 0)
       (effects (font (size 1.27 1.27)) (justify left bottom))
     )
-    (property "Sheetfile" "ANC_FF_Filter.kicad_sch" (at 105.41 59.0046 0)
+    (property "Sheetfile" "ANC_FF_Filter.kicad_sch" (at 105.41 67.8946 0)
       (effects (font (size 1.27 1.27)) (justify left top))
     )
-    (pin "QOP1" input (at 105.41 53.34 180)
-      (effects (font (size 1.27 1.27)) (justify left))
-    )
-    (pin "GNDA" input (at 105.41 55.88 180)
-      (effects (font (size 1.27 1.27)) (justify left))
-    )
-    (pin "IOP1" input (at 105.41 50.8 180)
-      (effects (font (size 1.27 1.27)) (justify left))
-    )
-    (pin "QMIC" input (at 105.41 48.26 180)
+    (pin "QOP1" input (at 105.41 62.23 180)
+      (effects (font (size 1.27 1.27)) (justify left))
+    )
+    (pin "GNDA" input (at 105.41 64.77 180)
+      (effects (font (size 1.27 1.27)) (justify left))
+    )
+    (pin "IOP1" input (at 105.41 59.69 180)
+      (effects (font (size 1.27 1.27)) (justify left))
+    )
+    (pin "QMIC" input (at 105.41 57.15 180)
       (effects (font (size 1.27 1.27)) (justify left))
     )
@@
     )
   )
-  (sheet (at 105.41 63.5) (size 29.21 12.7) (fields_autoplaced)
+  (sheet (at 105.41 72.39) (size 29.21 12.7) (fields_autoplaced)
     (stroke (width 0.1524) (type solid))
     (fill (color 0 0 0 0.0000))
-    (property "Sheetname" "filter_L" (at 105.41 62.7884 0)
+    (property "Sheetname" "filter_L" (at 105.41 71.6784 0)
       (effects (font (size 1.27 1.27)) (justify left bottom))
     )
-    (property "Sheetfile" "ANC_FF_Filter.kicad_sch" (at 105.41 76.7846 0)
+    (property "Sheetfile" "ANC_FF_Filter.kicad_sch" (at 105.41 85.6746 0)
       (effects (font (size 1.27 1.27)) (justify left top))
     )
-    (pin "QOP1" input (at 105.41 71.12 180)
-      (effects (font (size 1.27 1.27)) (justify left))
-    )
-    (pin "GNDA" input (at 105.41 73.66 180)
-      (effects (font (size 1.27 1.27)) (justify left))
-    )
-    (pin "IOP1" input (at 105.41 68.58 180)
-      (effects (font (size 1.27 1.27)) (justify left))
-    )
-    (pin "QMIC" input (at 105.41 66.04 180)
-      (effects (font (size 1.27 1.27)) (justify left))
-    )
+    (pin "QOP1" input (at 105.41 80.01 180)
+      (effects (font (size 1.27 1.27)) (justify left))
+    )
+    (pin "GNDA" input (at 105.41 82.55 180)
+      (effects (font (size 1.27 1.27)) (justify left))
+    )
+    (pin "IOP1" input (at 105.41 77.47 180)
+      (effects (font (size 1.27 1.27)) (justify left))
+    )
+    (pin "QMIC" input (at 105.41 74.93 180)
+      (effects (font (size 1.27 1.27)) (justify left))
+    )
