File: electronics/right/right.kicad_pcb (KiCad board)
At the start: 2 copper layers, 50.6 x 52.3 mm, 38 parts, among them J5 programming, J6 Batt, SW1 jog stick, SW2 Volume up, SW3 Volume down, U1 ATtiny441-M, U2 AP22814AW5, Y1 8Mhz

Commit message: all pcbs done and ordered
Changed lines of the file:
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@@
       (outputformat 1)
       (mirror false)
-      (drillshape 1)
+      (drillshape 0)
       (scaleselection 1)
-      (outputdirectory "")
+      (outputdirectory "right fab/")
     )
   )
@@
     (pad "2" smd roundrect (at 0.5 1.325 359.9) (size 0.6 1.55) (layers "F.Cu" "F.Paste" "F.Mask") (roundrect_rratio 0.25)
       (net 2 "GND") (pinfunction "Pin_2") (pintype "passive"))
-    (pad "MP" smd roundrect (at -1.8 -1.2 359.9) (size 1.2 1.8) (layers "F.Cu" "F.Paste" "F.Mask") (roundrect_rratio 0.208333)
+    (pad "MP" smd roundrect (at -1.8 -1.2 359.9) (size 1.2 1.8) (layers "F.Cu" "F.Paste" "F.Mask") (roundrect_rratio 0.2083333333)
       (net 2 "GND") (pinfunction "MP") (pintype "passive"))
-    (pad "MP" smd roundrect (at 1.8 -1.2 359.9) (size 1.2 1.8) (layers "F.Cu" "F.Paste" "F.Mask") (roundrect_rratio 0.208333)
+    (pad "MP" smd roundrect (at 1.8 -1.2 359.9) (size 1.2 1.8) (layers "F.Cu" "F.Paste" "F.Mask") (roundrect_rratio 0.2083333333)
       (net 2 "GND") (pinfunction "MP") (pintype "passive"))
     (model "C:/Users/alexl/projects/headphones/electronics/components/BM02B-SRSS-TB-LF--SN---3DModel-STEP-56544 v2.step"
@@
     (property "ki_keywords" "AVR 8bit Microcontroller tinyAVR")
     (attr smd)
-    (fp_text reference "U1" (at -3.475 -1.1 -180) (layer "B.SilkS")
+    (fp_text reference "U1" (at -3.475 -1.1) (layer "B.SilkS")
         (effects (font (size 1 1) (thickness 0.15)) (justify mirror))
     )
@@
     (fp_line (start 2 2) (end 2 -2)
       (stroke (width 0.1) (type solid)) (layer "B.Fab"))
-    (pad "" smd roundrect (at -0.65 -0.65 270) (size 1.05 1.05) (layers "B.Paste") (roundrect_rratio 0.238095))
-    (pad "" smd roundrect (at -0.65 0.65 270) (size 1.05 1.05) (layers "B.Paste") (roundrect_rratio 0.238095))
-    (pad "" smd roundrect (at 0.65 -0.65 270) (size 1.05 1.05) (layers "B.Paste") (roundrect_rratio 0.238095))
-    (pad "" smd roundrect (at 0.65 0.65 270) (size 1.05 1.05) (layers "B.Paste") (roundrect_rratio 0.238095))
+    (pad "" smd roundrect (at -0.65 -0.65 270) (size 1.05 1.05) (layers "B.Paste") (roundrect_rratio 0.2380952381))
+    (pad "" smd roundrect (at -0.65 0.65 270) (size 1.05 1.05) (layers "B.Paste") (roundrect_rratio 0.2380952381))
+    (pad "" smd roundrect (at 0.65 -0.65 270) (size 1.05 1.05) (layers "B.Paste") (roundrect_rratio 0.2380952381))
+    (pad "" smd roundrect (at 0.65 0.65 270) (size 1.05 1.05) (layers "B.Paste") (roundrect_rratio 0.2380952381))
     (pad "1" smd roundrect (at -1.925 1 270) (size 0.85 0.25) (layers "B.Cu" "B.Paste" "B.Mask") (roundrect_rratio 0.25)
       (net 7 "/SCK") (pinfunction "PA4") (pintype "bidirectional"))
@@
     (pad "21" smd rect (at 0 0 270) (size 2.6 2.6) (layers "B.Cu" "B.Mask")
       (net 2 "GND") (pinfunction "GND") (pintype "passive"))
-    (model "${KICAD6_3DMODEL_DIR}/Package_DFN_QFN.3dshapes/QFN-20-1EP_4x4mm_P0.5mm_EP2.6x2.6mm.wrl"
+    (model "${KICAD7_3DMODEL_DIR}/Package_DFN_QFN.3dshapes/QFN-20-1EP_4x4mm_P0.5mm_EP2.5x2.5mm.wrl"
       (offset (xyz 0 0 0))
       (scale (xyz 1 1 1))
@@
     (property "ki_description" "Two pin crystal, small symbol")
     (property "ki_keywords" "quartz ceramic resonator oscillator")
-    (attr smd)
+    (attr smd exclude_from_pos_files)
     (fp_text reference "Y1" (at 1.6 -2.7) (layer "B.SilkS")
         (effects (font (size 1 1) (thickness 0.15)) (justify mirror))
@@
   (gr_line (start 35.8073 70.095399) (end 37.936002 63.711349)
     (stroke (width 0.2) (type solid)) (layer "Edge.Cuts"))
-  (gr_line (start 38.527827 61.941911) (end 41.425572 53.261303)
-    (stroke (width 0.2) (type solid)) (layer "Edge.Cuts"))
   (gr_line (start 38.674271 100.57265) (end 42.415401 102.646392)
     (stroke (width 0.2) (type solid)) (layer "Edge.Cuts"))
@@
   (gr_line (start 38.527827 61.941911) (end 37.694462 61.844304)
     (stroke (width 0.2) (type default)) (layer "Edge.Cuts"))
+  (gr_line (start 38.527827 61.941911) (end 41.425572 53.261303)
+    (stroke (width 0.2) (type solid)) (layer "Edge.Cuts"))
   (gr_line (start 30.934097 92.704216) (end 38.63133 96.970863)
     (stroke (width 0.2) (type solid)) (layer "Edge.Cuts"))
@@
     (effects (font (size 1 1) (thickness 0.15)) (justify left bottom))
   )
-  (gr_text "ALM" (at 30.5 57.5 265) (layer "F.SilkS")
-    (effects (font (face "Imperial Black") (size 5 5) (thickness 0.3) bold) (justify left bottom))
+  (gr_text "ALM" (at 30.9 58.5 265) (layer "F.SilkS")
+    (effects (font (face "Madeon Runes Bold") (size 5 5) (thickness 0.3) bold) (justify left bottom))
     (render_cache "ALM" 265
       (polygon
         (pts
-          (xy 32.113505 61.575009)          (xy 31.005212 61.478046)          (xy 31.319517 57.885523)          (xy 32.399829 57.980038)
-          (xy 36.097262 60.668242)          (xy 35.985717 61.943205)          (xy 32.313498 59.289079)
+          (xy 36.415144 61.710093)          (xy 32.08862 58.60399)          (xy 31.746765 58.574082)          (xy 31.474183 61.68971)
+          (xy 31.987574 61.734626)          (xy 32.199062 59.317307)          (xy 36.060641 62.090973)          (xy 36.379382 62.11886)
         )
       )
       (polygon
         (pts
-          (xy 31.717256 65.781883)          (xy 30.636944 65.687368)          (xy 30.951249 62.094845)          (xy 32.059542 62.191808)
-          (xy 31.859549 64.477738)          (xy 32.722409 64.059199)          (xy 32.879508 62.263546)          (xy 33.987801 62.360509)
-          (xy 33.889029 63.489484)          (xy 35.936863 62.501609)          (xy 35.825318 63.776571)          (xy 33.776845 64.771745)
-          (xy 33.673496 65.953032)          (xy 32.565203 65.856069)          (xy 32.610119 65.342678)
+          (xy 36.294765 63.086031)          (xy 35.971158 63.057719)          (xy 34.01782 64.002374)          (xy 34.114677 62.895297)
+          (xy 33.601285 62.850382)          (xy 33.477607 64.264033)          (xy 31.691789 65.115466)          (xy 31.902958 62.701797)
+          (xy 31.389566 62.656881)          (xy 31.116984 65.77251)          (xy 31.452757 65.801886)          (xy 33.42556 64.858934)
+          (xy 33.328703 65.96601)          (xy 33.842095 66.010926)          (xy 33.965773 64.597275)          (xy 36.259322 63.491147)
         )
       )
       (polygon
         (pts
-          (xy 32.970417 67.711951)          (xy 35.56785 66.719447)          (xy 35.459072 67.962779)          (xy 34.190306 68.438972)
-          (xy 35.356575 69.134333)          (xy 35.252693 70.321703)          (xy 30.269634 69.885741)          (xy 30.347076 69.000586)
-          (xy 32.706893 69.000586)          (xy 33.006168 69.026769)          (xy 32.86281 68.9419)          (xy 32.706893 69.000586)
-          (xy 30.347076 69.000586)          (xy 30.373516 68.698372)          (xy 31.642814 68.216096)          (xy 30.476013 67.526818)
-          (xy 30.584791 66.283486)
+          (xy 31.372034 66.808626)          (xy 31.381766 66.809477)          (xy 33.38092 68.255617)          (xy 35.609337 67.179342)
+          (xy 35.93416 67.20776)          (xy 35.898611 67.614093)          (xy 33.856175 68.596311)          (xy 35.696383 69.925571)
+          (xy 35.658279 70.361102)          (xy 30.75308 69.931953)          (xy 30.789907 69.511021)          (xy 30.829953 69.491557)
+          (xy 31.996649 69.491557)          (xy 34.527108 69.712944)          (xy 33.328873 68.850518)          (xy 31.996649 69.491557)
+          (xy 30.829953 69.491557)          (xy 32.852507 68.508501)          (xy 30.994689 67.170345)          (xy 31.028962 66.778611)
         )
       )
